File: Electronics/Circuit-PCB.brd (EAGLE design)
At the start: 62.2 x 68.2 mm, 18 parts

Commit message: Updated all electronics files
Parts:
- moved SW1 53.9 mm to (12.7, 8.89), turned to 0 degrees
- moved D1 39.7 mm to (43.2, 52.1)
- moved D7 38.8 mm to (25.4, 17.8), turned to 180 degrees
- moved R1 38.6 mm to (44.5, 44.5)
- moved D6 38.1 mm to (25.4, 22.9), turned to 180 degrees
- moved D5 36.9 mm to (25.4, 29.2), turned to 180 degrees
- moved SW2 30.2 mm to (24.1, 50.8)
- moved R2 26.2 mm to (24.1, 12.7)
- moved JP4 17.8 mm to (3.81, 40.6), turned to 270 degrees
- moved R4 17.0 mm to (24.1, 36.8), turned to 90 degrees
- moved G1 16.5 mm to (19.1, 61.0), turned to 180 degrees
- moved R3 15.9 mm to (24.1, 43.2), turned to 90 degrees
- moved JP3 12.7 mm to (3.81, 17.8), turned to 270 degrees
- moved R7 6.35 mm to (35.6, 29.2)
- moved R6 2.54 mm to (35.6, 22.9)
Connections:
- net N$13: now also JP5.1
Routing:
- net N$7: track 87.4 -> 7.94 mm, vias 2 -> 0
- net N$9: track 63.9 -> 7.94 mm, vias 2 -> 0
- net N$4: track 63.5 -> 7.94 mm, vias 2 -> 0
- net N$5: track 89.4 -> 39.7 mm, vias 1 -> 0
- net N$6: track 35.5 -> 3.67 mm
- net N$3: track 35.7 -> 6.48 mm, vias 2 -> 0
- net N$2: track 41.4 -> 14.4 mm
- net N$14: track 15.1 -> 28.5 mm, vias 0 -> 1
- net N$1: track 69.0 -> 62.5 mm
- net N$13: track 72.3 -> 67.2 mm
- net N$11: track 15.6 -> 18.2 mm
- net N$10: track 15.6 -> 16.6 mm
Other:
- board size 62.2 x 68.2 mm -> 57.1 x 68.2 mm
